Commit message: fix [not working] start of aruco integration

File: eagerx_interbotix/solid/assets/box.urdf (robot description, URDF)
Before this commit: robot box, 1 links, 0 joints
Links:
- link baseLink: mass 0.358 -> 0.047; geometry collision box size=0.1 0.1 0.1; visual box size=0.1 0.1 0.1

File: eagerx_interbotix/solid/assets/box_goal.urdf (robot description, URDF)
Before this commit: robot box, 1 links, 0 joints
Links:
- link baseLink: geometry visual box size=0.1 0.1 0.1
