Commit message: add domain randomisation shadows and colours

File: eagerx_interbotix/solid/assets/surface.urdf (robot description, URDF)
Before this commit: robot box, 1 links, 0 joints
Links:
- link baseLink: geometry visual box size=2.0 2.0 0.01

Commit message: fix: updates after experiments

File: eagerx_interbotix/solid/assets/surface.urdf (robot description, URDF)
Before this commit: robot box, 1 links, 0 joints
Links:
- link baseLink: geometry visual box size=5.0 5.0 0.01
